Commit message: feat: 添加 mid-360 仿真文件

File: urdf/livox_mid360.xacro (robot description, xacro)
@@ -4,10 +4,10 @@
   <xacro:property name="laser_min_range" value="0.1"/>
   <xacro:property name="laser_max_range" value="200.0"/>
-  <xacro:property name="ros_topic" value="scan"/>
+  <xacro:property name="ros_topic" value="/livox/lidar"/>
   <xacro:property name="samples" value="24000"/>
   <xacro:property name="downsample" value="1"/>
   <xacro:macro name="null_inertial">
     <inertial>
-      <mass value="0.1"/>
+      <mass value="0.001"/>
     <inertia ixx="0.01" ixy="0" ixz="0"
           iyy="0.01" iyz="0"
@@ -58,5 +58,5 @@
     </gazebo>
   </xacro:macro>
-  <xacro:macro name="Livox_Mid40" params="visualize:=True name:=livox">
+  <xacro:macro name="Livox_Mid360" params="visualize:=True name:=livox">
     <link name="${name}_base">
       <xacro:null_inertial/>
@@ -77,5 +77,5 @@
       <xacro:null_inertial/>
     </link>
-    <joint name="${name}_to_${name}_base_joint" type="fixed">
+    <joint name="${name}_to_livox_base_joint" type="fixed">
       <parent link="${name}_base"/>
       <child link="${name}"/>
@@ -84,6 +84,6 @@
     <xacro:Livox_Mid_gazebo_sensor name="${name}" visualize="${visualize}"/>
   </xacro:macro>
-    <xacro:Livox_Mid40 name="livox"/>
-  <xacro:include filename="$(find livox_laser_simulation)/urdf/standardrobots_oasis300.xacro"/>
-  <xacro:link_oasis name="oasis"/>
+    <!--xacro:Livox_Mid40 name="livox"/-->
+  <!--xacro:include filename="$(find livox_laser_simulation)/urdf/standardrobots_oasis300.xacro"/>
+  <xacro:link_oasis name="oasis"/-->
 </robot>
