Commit message: feat: 实现 husky 携带 mid-360

File: urdf/husky_mid360_IMU_platform.xacro (robot description, xacro)
@@ -1,7 +1,6 @@
 <?xml version="1.0"?>
 <robot xmlns:xacro="http://www.ros.org/wiki/xacro" name="example">
-  <!-- Base Footprint -->
-  <link name="base_link" />
-  <xacro:macro name="LivoxMid360_IMU_Plantform" params="name:=mid360_imu_plantform parent_link_name:=base_link x:=0.0 y:=0.0 z:=0.05 r:=0.0 p:=0.0 yaw:=0.0">
+  <xacro:include filename="$(find husky_description)/urdf/husky.urdf.xacro"/>
+  <xacro:macro name="LivoxMid360_IMU_Plantform" params="name:=mid360_imu_plantform parent_link_name:=base_link x:=0.0 y:=0.0 z:=0.2 r:=0.0 p:=0.0 yaw:=0.0">
       <joint name="${name}_joint" type="fixed" >
         <parent link="${parent_link_name}" />
@@ -102,5 +101,3 @@
       <origin rpy="0 0 0" xyz="0.0 0.0 0.0"/>
     </joint>
-  <!--xacro:include filename="$(find livox_laser_simulation)/urdf/standardrobots_oasis300.xacro"/-->
-  <!--xacro:link_oasis name="oasis"/-->
 </robot>

File: urdf/livox_mid360.xacro (robot description, xacro)
@@ -80,5 +80,5 @@
       <parent link="${name}_base"/>
       <child link="${name}"/>
-      <origin rpy="0 0 0" xyz="0.0 1.0 0.2"/>
+      <origin rpy="0 0 0" xyz="0.0 0.0 0.35"/>
     </joint>
     <xacro:Livox_Mid_gazebo_sensor name="${name}" visualize="${visualize}"/>

Commit message: fix: 使 rvix 成功显示车体模型

File: urdf/husky_mid360_IMU_platform.xacro (robot description, xacro)
@@ -89,15 +89,15 @@
   </xacro:macro>
   <xacro:LivoxMid360_IMU_Plantform name="mid360_imu_plantform"/>
-  <link name="example::base_link" />
-  <link name="laser_livox" />
-    <joint name="base_link_to_example_base_link_joint" type="fixed">
+  <!--link name="example::base_link" /-->
+  <!--link name="laser_livox" /-->
+    <!--joint name="base_link_to_example_base_link_joint" type="fixed">
       <parent link="base_link"/>
       <child link="example::base_link"/>
       <origin rpy="0 0 0" xyz="0.0 0.0 0.0"/>
-    </joint>
-    <joint name="base_link_to_laser_livox_joint" type="fixed">
+    </joint-->
+    <!--joint name="base_link_to_laser_livox_joint" type="fixed">
       <parent link="base_link"/>
       <child link="laser_livox"/>
       <origin rpy="0 0 0" xyz="0.0 0.0 0.0"/>
-    </joint>
+    </joint-->
 </robot>
